Commit message: revive this repo...

File: src/dorna2/dorna2/urdf/dorna.urdf (robot description, URDF)
Before this commit: robot dorna, 6 links, 5 joints
Links:
- removed link dorna_1_link
- removed link dorna_2_link
- removed link dorna_3_link
- removed link dorna_4_link
- removed link dorna_5_link
- removed link dorna_base_link
- added link PREFIX_dorna_1_link, mass 1.579; collision mesh filename=package://dorna2/meshes/j0_c.stl scale=0.01 0.01 0.01; visual mesh filename=package://dorna2/meshes/j0_c.stl scale=0.01 0.01 0.01
- added link PREFIX_dorna_2_link, mass 0.709; collision mesh filename=package://dorna2/meshes/j1_c.stl scale=0.01 0.01 0.01; visual mesh filename=package://dorna2/meshes/j1_c.stl scale=0.01 0.01 0.01
- added link PREFIX_dorna_3_link, mass 0.501; collision mesh filename=package://dorna2/meshes/j2_c.stl scale=0.01 0.01 0.01; visual mesh filename=package://dorna2/meshes/j2_c.stl scale=0.01 0.01 0.01
- added link PREFIX_dorna_4_link, mass 0.075; collision mesh filename=package://dorna2/meshes/j3_c.stl scale=0.01 0.01 0.01; visual mesh filename=package://dorna2/meshes/j3_c.stl scale=0.01 0.01 0.01
- added link PREFIX_dorna_5_link, mass 0.042; collision mesh filename=package://dorna2/meshes/j4_c.stl scale=0.01 0.01 0.01; visual mesh filename=package://dorna2/meshes/j4_c.stl scale=0.01 0.01 0.01
- added link PREFIX_dorna_base_link, mass 0.848; collision mesh filename=package://dorna2/meshes/base_v8.stl scale=0.01 0.01 0.01; visual mesh filename=package://dorna2/meshes/base_v8.stl scale=0.01 0.01 0.01
Joints:
- removed joint dorna_axis_1_joint
- removed joint dorna_axis_2_joint
- removed joint dorna_axis_3_joint
- removed joint dorna_axis_4_joint
- removed joint dorna_axis_5_joint
- added joint PREFIX_dorna_axis_1_joint: type revolute, parent PREFIX_dorna_base_link, child PREFIX_dorna_1_link, origin xyz=0 0 0 rpy=0 0 0, axis 0 0 1, limit lower=-3.49 upper=3.05433 effort=50 velocity=5.236
- added joint PREFIX_dorna_axis_2_joint: type revolute, parent PREFIX_dorna_1_link, child PREFIX_dorna_2_link, origin xyz=0.095 0 0.20603 rpy=3.14159265359 0 0, axis 0 1 0, limit lower=-3.05433 upper=2.79253 effort=50 velocity=2.618
- added joint PREFIX_dorna_axis_3_joint: type revolute, parent PREFIX_dorna_2_link, child PREFIX_dorna_3_link, origin xyz=0.20327 0 0 rpy=0 0 0, axis 0 1 0, limit lower=-2.26893 upper=2.26893 effort=50 velocity=2.618
- added joint PREFIX_dorna_axis_4_joint: type continuous, parent PREFIX_dorna_3_link, child PREFIX_dorna_4_link, origin xyz=0.15245 0 0 rpy=0 0 0, axis 0 1 0, limit lower=0 upper=6.28318530718 effort=50 velocity=5.236
- added joint PREFIX_dorna_axis_5_joint: type continuous, parent PREFIX_dorna_4_link, child PREFIX_dorna_5_link, origin xyz=0.0 0.0 0.0 rpy=0 0 0, axis 1 0 0, limit lower=0 upper=6.28318530718 effort=50 velocity=5.236
